File: hardware/dewcontrollerQ150/dewcontrollerQ150.kicad_sch (KiCad schematic)
At the start: 13 parts, among them J1 12V Power, J2 Dew Heater, J3 SHT45 Sensor, Q1 FQP 30N06L, U1 XIAO-ESP32-C3-DIP, U2 Buck_12V_5V

Commit message: V0.51 updated KiCAD schematic with S3
Parts:
- removed U1: XIAO-ESP32-C3-DIP, Module:MOUDLE14P-XIAO-DIP-SMD, symbol Seeed_Studio_XIAO_Series:XIAO-ESP32-C3-DIP
- added U3: XIAO-ESP32-S3-DIP, RF_Module:MCU_Seeed_ESP32C3, symbol Seeed_Studio_XIAO_Series:XIAO-ESP32-S3-DIP
Connections:
- net 3.3V: now also U3.12 (VCC_3V3)
- net 5V: now also U3.14 (VBUS)
- net GND: now also U3.13 (GND)
- net SCL: now also U3.6 (GPIO9/D5/I2C_SCL)
- net SDA: now also U3.5 (GPIO5/D4/I2C_SDA)
- net at R1.1: now also U3.9 (GPIO7/D8/A8/SCK)
Other:
- moved on the sheet: C3, C4, J2, Q1, R1, R2

Commit message: v0.6 tidy up code
Parts:
- C1: footprint (none) -> Capacitor_THT:CP_Radial_D10.0mm_P5.00mm
- C2, C3, C4: footprint (none) -> Capacitor_THT:C_Disc_D5.1mm_W3.2mm_P5.00mm
- J1, J2: footprint (none) -> Connector_JST:JST_XH_B2B-XH-A_1x02_P2.50mm_Vertical
- J3: footprint (none) -> Connector_JST:JST_XH_B4B-XH-A_1x04_P2.50mm_Vertical
- Q1: footprint (none) -> Package_TO_SOT_THT:TO-218-3_Vertical
- R1, R2, R3: footprint (none) -> Resistor_THT:R_Axial_DIN0207_L6.3mm_D2.5mm_P7.62mm_Horizontal
Changed lines of the file:
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@@
-	)
-	(junction
-		(at 209.55 93.98)
-		(diameter 0)
-		(color 0 0 0 0)
 	)
 	(junction
@@
 		(pts
 			(xy 92.71 73.66) (xy 100.33 73.66)
-		)
-		(stroke
-			(width 0)
-			(type default)
-		)
-	)
-	(wire
-		(pts
-			(xy 209.55 93.98) (xy 204.47 93.98)
 		)
 		(stroke
@@
 	(label "3.3V"
 		(at 102.87 120.65 180)
-		(effects
-			(font
-				(size 1.27 1.27)
-			)
-			(justify right bottom)
-		)
-	)
-	(label "+Heater"
-		(at 209.55 93.98 180)
 		(effects
 			(font
@@
 			)
 		)
-		(property "Footprint" ""
+		(property "Footprint" "Package_TO_SOT_THT:TO-218-3_Vertical"
 			(at 212.09 109.22 0)
 			(effects
@@
 			)
 		)
-		(property "Footprint" ""
+		(property "Footprint" "Capacitor_THT:C_Disc_D5.1mm_W3.2mm_P5.00mm"
 			(at 182.5752 100.33 0)
 			(effects
@@
 			)
 		)
-		(property "Footprint" ""
+		(property "Footprint" "Capacitor_THT:CP_Radial_D10.0mm_P5.00mm"
 			(at 98.7552 90.17 0)
 			(effects
@@
 			)
 		)
-		(property "Footprint" ""
+		(property "Footprint" "Resistor_THT:R_Axial_DIN0207_L6.3mm_D2.5mm_P7.62mm_Horizontal"
 			(at 112.522 66.04 90)
 			(effects
@@
 			)
 		)
-		(property "Footprint" ""
+		(property "Footprint" "Capacitor_THT:C_Disc_D5.1mm_W3.2mm_P5.00mm"
 			(at 105.1052 90.17 0)
 			(effects
@@
 			)
 		)
-		(property "Footprint" ""
+		(property "Footprint" "Connector_JST:JST_XH_B2B-XH-A_1x02_P2.50mm_Vertical"
 			(at 87.63 73.66 0)
 			(effects
@@
 			)
 		)
-		(property "Footprint" ""
+		(property "Footprint" "Resistor_THT:R_Axial_DIN0207_L6.3mm_D2.5mm_P7.62mm_Horizontal"
 			(at 184.15 113.538 90)
 			(effects
@@
 			)
 		)
-		(property "Footprint" ""
+		(property "Footprint" "Connector_JST:JST_XH_B2B-XH-A_1x02_P2.50mm_Vertical"
 			(at 214.63 93.98 0)
 			(effects
@@
 			)
 		)
-		(property "Footprint" ""
+		(property "Footprint" "Capacitor_THT:C_Disc_D5.1mm_W3.2mm_P5.00mm"
 			(at 192.7352 100.33 0)
 			(effects
@@
 			)
 		)
-		(property "Footprint" ""
+		(property "Footprint" "Resistor_THT:R_Axial_DIN0207_L6.3mm_D2.5mm_P7.62mm_Horizontal"
 			(at 191.262 120.65 90)
 			(effects
@@
 			)
 		)
-		(property "Footprint" ""
+		(property "Footprint" "Connector_JST:JST_XH_B4B-XH-A_1x04_P2.50mm_Vertical"
 			(at 93.98 118.11 0)
 			(effects

Commit message: V1.2 PCB fixed ESP32S3 and FQP30N06 footprints
Parts:
- Q1: footprint Package_TO_SOT_THT:TO-218-3_Vertical -> Package_TO_SOT_THT:TO-220-3_Vertical
Changed lines of the file:
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@@
 		(title "Dew Heater Controller for Q150")
 		(date "2026-01-27")
-		(rev "0.1")
+		(rev "B")
 		(company "Mark Pinnuck")
 	)
@@
 			)
 		)
-		(property "Footprint" "Package_TO_SOT_THT:TO-218-3_Vertical"
+		(property "Footprint" "Package_TO_SOT_THT:TO-220-3_Vertical"
 			(at 212.09 109.22 0)
 			(effects

Commit message: v1.2b Changed esp32-S3 to correct footprint
Parts:
- U3: footprint RF_Module:MCU_Seeed_ESP32C3 -> Seeed Studio XIAO Series Library:XIAO-ESP32S3-DIP
Changed lines of the file:
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@@
 			)
 		)
-		(property "Footprint" "RF_Module:MCU_Seeed_ESP32C3"
+		(property "Footprint" "Seeed Studio XIAO Series Library:XIAO-ESP32S3-DIP"
 			(at 133.858 119.38 0)
 			(effects
